File: circuit/TEMPSENSE.kicad_pcb (KiCad board)
At the start: 2 copper layers, 47 x 40.6 mm, 5 parts, among them U1 MAX31855, U2 MAX31855, U3 MAX31855, U4 MAX31855, U5 FT232H

Commit message: updates schematic and pcb
Connections:
- net MISO renamed CIPO
